Commit message: change repo title

File: urdf/robotiq_arg2f_140_model/robotiq_arg2f.xacro (robot description, xacro)
@@ -11,5 +11,5 @@
         <origin xyz="0 0 0" rpy="0 0 0" />
         <geometry>
-          <mesh filename="package://shallow_depth_insertion_v2/meshes/robotiq_arg2f_140_model/visual/robotiq_arg2f_base_link.stl" />
+          <mesh filename="package://shallow_depth_insertion/meshes/robotiq_arg2f_140_model/visual/robotiq_arg2f_base_link.stl" />
         </geometry>
         <material name="">
@@ -20,5 +20,5 @@
         <origin xyz="0 0 0" rpy="0 0 0" />
         <geometry>
-          <mesh filename="package://shallow_depth_insertion_v2/meshes/robotiq_arg2f_140_model/collision/robotiq_arg2f_base_link.stl" />
+          <mesh filename="package://shallow_depth_insertion/meshes/robotiq_arg2f_140_model/collision/robotiq_arg2f_base_link.stl" />
         </geometry>
       </collision>

File: urdf/robotiq_arg2f_140_model/robotiq_arg2f_140_model.xacro (robot description, xacro)
@@ -1,5 +1,5 @@
 <?xml version="1.0"?>
 <robot name="robotiq_arg2f_140_model" xmlns:xacro="http://ros.org/wiki/xacro">
-  <xacro:include filename="$(find shallow_depth_insertion_v2)/urdf/robotiq_arg2f_140_model/robotiq_arg2f_140_model_macro.xacro" />
+  <xacro:include filename="$(find shallow_depth_insertion)/urdf/robotiq_arg2f_140_model/robotiq_arg2f_140_model_macro.xacro" />
   <xacro:robotiq_arg2f_140 prefix=""/>
 </robot>

File: urdf/robotiq_arg2f_140_model/robotiq_arg2f_140_model_macro.xacro (robot description, xacro)
@@ -1,5 +1,5 @@
 <?xml version="1.0"?>
 <robot xmlns:xacro="http://ros.org/wiki/xacro">
-  <xacro:include filename="$(find shallow_depth_insertion_v2)/urdf/robotiq_arg2f_140_model/robotiq_arg2f_transmission.xacro" />
+  <xacro:include filename="$(find shallow_depth_insertion)/urdf/robotiq_arg2f_140_model/robotiq_arg2f_transmission.xacro" />
   <xacro:macro name="outer_knuckle" params="prefix fingerprefix stroke">
     <link name="${prefix}${fingerprefix}_outer_knuckle">
@@ -18,5 +18,5 @@
         <origin xyz="0 0 0" rpy="0 0 0" />
         <geometry>
-          <mesh filename="package://shallow_depth_insertion_v2/meshes/robotiq_arg2f_140_model/visual/robotiq_arg2f_${stroke}_outer_knuckle.stl" />
+          <mesh filename="package://shallow_depth_insertion/meshes/robotiq_arg2f_140_model/visual/robotiq_arg2f_${stroke}_outer_knuckle.stl" />
         </geometry>
         <material name="">
@@ -27,5 +27,5 @@
         <origin xyz="0 0 0" rpy="0 0 0" />
         <geometry>
-          <mesh filename="package://shallow_depth_insertion_v2/meshes/robotiq_arg2f_140_model/collision/robotiq_arg2f_${stroke}_outer_knuckle.stl" />
+          <mesh filename="package://shallow_depth_insertion/meshes/robotiq_arg2f_140_model/collision/robotiq_arg2f_${stroke}_outer_knuckle.stl" />
         </geometry>
       </collision>
@@ -48,5 +48,5 @@
         <origin xyz="0 0 0" rpy="0 0 0" />
         <geometry>
-          <mesh filename="package://shallow_depth_insertion_v2/meshes/robotiq_arg2f_140_model/visual/robotiq_arg2f_${stroke}_outer_finger.stl" />
+          <mesh filename="package://shallow_depth_insertion/meshes/robotiq_arg2f_140_model/visual/robotiq_arg2f_${stroke}_outer_finger.stl" />
         </geometry>
         <material name="">
@@ -57,5 +57,5 @@
         <origin xyz="0 0 0" rpy="0 0 0" />
         <geometry>
-          <mesh filename="package://shallow_depth_insertion_v2/meshes/robotiq_arg2f_140_model/collision/robotiq_arg2f_${stroke}_outer_finger.stl" />
+          <mesh filename="package://shallow_depth_insertion/meshes/robotiq_arg2f_140_model/collision/robotiq_arg2f_${stroke}_outer_finger.stl" />
         </geometry>
       </collision>
@@ -78,5 +78,5 @@
         <origin xyz="0 0 0" rpy="0 0 0" />
         <geometry>
-          <mesh filename="package://shallow_depth_insertion_v2/meshes/robotiq_arg2f_140_model/visual/robotiq_arg2f_${stroke}_inner_knuckle.stl" />
+          <mesh filename="package://shallow_depth_insertion/meshes/robotiq_arg2f_140_model/visual/robotiq_arg2f_${stroke}_inner_knuckle.stl" />
         </geometry>
         <material name="">
@@ -87,5 +87,5 @@
         <origin xyz="0 0 0" rpy="0 0 0" />
         <geometry>
-          <mesh filename="package://shallow_depth_insertion_v2/meshes/robotiq_arg2f_140_model/collision/robotiq_arg2f_${stroke}_inner_knuckle.stl" />
+          <mesh filename="package://shallow_depth_insertion/meshes/robotiq_arg2f_140_model/collision/robotiq_arg2f_${stroke}_inner_knuckle.stl" />
         </geometry>
       </collision>
@@ -108,5 +108,5 @@
         <origin xyz="0 0 0" rpy="0 0 0" />
         <geometry>
-          <mesh filename="package://shallow_depth_insertion_v2/meshes/robotiq_arg2f_140_model/visual/robotiq_arg2f_${stroke}_inner_finger.stl" />
+          <mesh filename="package://shallow_depth_insertion/meshes/robotiq_arg2f_140_model/visual/robotiq_arg2f_${stroke}_inner_finger.stl" />
         </geometry>
         <material name="">
@@ -117,5 +117,5 @@
         <origin xyz="0 0 0" rpy="0 0 0" />
         <geometry>
-          <mesh filename="package://shallow_depth_insertion_v2/meshes/robotiq_arg2f_140_model/collision/robotiq_arg2f_${stroke}_inner_finger.stl" />
+          <mesh filename="package://shallow_depth_insertion/meshes/robotiq_arg2f_140_model/collision/robotiq_arg2f_${stroke}_inner_finger.stl" />
         </geometry>
       </collision>
@@ -194,5 +194,5 @@
     </joint>
   </xacro:macro>
-  <xacro:include filename="$(find shallow_depth_insertion_v2)/urdf/robotiq_arg2f_140_model/robotiq_arg2f.xacro" />
+  <xacro:include filename="$(find shallow_depth_insertion)/urdf/robotiq_arg2f_140_model/robotiq_arg2f.xacro" />
   <xacro:macro name="finger_joint" params="prefix">
     <joint name="${prefix}finger_joint" type="revolute">

File: urdf/robotiq_ft_sensor/robotiq_ft300.urdf.xacro (robot description, xacro)
@@ -30,5 +30,5 @@
                 <origin xyz="0 0 0" rpy="0 0 0" />
                 <geometry>
-                    <mesh filename="package://shallow_depth_insertion_v2/meshes/robotiq_ft_sensor/visual/robotiq_ft300.STL"/>
+                    <mesh filename="package://shallow_depth_insertion/meshes/robotiq_ft_sensor/visual/robotiq_ft300.STL"/>
                 </geometry>
                 <material name="Robotiq-Black">
@@ -39,5 +39,5 @@
                 <origin xyz="0 0 0" rpy="0 0 0" />
                 <geometry>
-                    <mesh filename="package://shallow_depth_insertion_v2/meshes/robotiq_ft_sensor/collision/robotiq_ft300.STL"/>
+                    <mesh filename="package://shallow_depth_insertion/meshes/robotiq_ft_sensor/collision/robotiq_ft300.STL"/>
                 </geometry>
             </collision>
@@ -48,5 +48,5 @@
                 <origin xyz="0 0 0" rpy="0 0 0" />
                 <geometry>
-                    <mesh filename="package://shallow_depth_insertion_v2/meshes/robotiq_ft_sensor/visual/mountings/robotiq_ft300-G-062-COUPLING_G-50-4M6-1D6_20181119.STL"/>
+                    <mesh filename="package://shallow_depth_insertion/meshes/robotiq_ft_sensor/visual/mountings/robotiq_ft300-G-062-COUPLING_G-50-4M6-1D6_20181119.STL"/>
                 </geometry>
                 <material name="Robotiq-Grey">
@@ -57,5 +57,5 @@
                 <origin xyz="0 0 0" rpy="0 0 0" />
                 <geometry>
-                    <mesh filename="package://shallow_depth_insertion_v2/meshes/robotiq_ft_sensor/collision/mountings/robotiq_ft300-G-062-COUPLING_G-50-4M6-1D6_20181119.STL"/>
+                    <mesh filename="package://shallow_depth_insertion/meshes/robotiq_ft_sensor/collision/mountings/robotiq_ft300-G-062-COUPLING_G-50-4M6-1D6_20181119.STL"/>
                 </geometry>
             </collision>

File: urdf/robotiq_ft_sensor/robotiq_fts150.urdf.xacro (robot description, xacro)
@@ -18,5 +18,5 @@
                 <origin xyz="0 0 0" rpy="0 0 0" />
                 <geometry>
-                    <mesh filename="package://shallow_depth_insertion_v2/meshes/robotiq_ft_sensor/visual/robotiq_fts150.stl"/>
+                    <mesh filename="package://shallow_depth_insertion/meshes/robotiq_ft_sensor/visual/robotiq_fts150.stl"/>
                 </geometry>
                 <material name="black"/>
@@ -25,5 +25,5 @@
                 <origin xyz="0 0 0" rpy="0 0 0" />
                 <geometry>
-                    <mesh filename="package://shallow_depth_insertion_v2/meshes/robotiq_ft_sensor/collision/robotiq_fts150.stl"/>
+                    <mesh filename="package://shallow_depth_insertion/meshes/robotiq_ft_sensor/collision/robotiq_fts150.stl"/>
                 </geometry>
             </collision>

File: urdf/ur10.urdf.xacro (robot description, xacro)
@@ -5,6 +5,6 @@
   Contributers: Jimmy Da Silva, Ajit Krisshna N L, Muhammad Asif Rana
 -->
-  <xacro:include filename="$(find shallow_depth_insertion_v2)/urdf/ur.transmission.xacro" />
-  <xacro:include filename="$(find shallow_depth_insertion_v2)/urdf/ur.gazebo.xacro" />
+  <xacro:include filename="$(find shallow_depth_insertion)/urdf/ur.transmission.xacro" />
+  <xacro:include filename="$(find shallow_depth_insertion)/urdf/ur.gazebo.xacro" />
   <!-- Inertia parameters -->
   <xacro:property name="base_mass" value="4.0" />  <!-- This mass might be incorrect -->
@@ -62,13 +62,13 @@
       <visual>
         <geometry>
-          <mesh filename="package://shallow_depth_insertion_v2/meshes/ur10/visual/base.dae"/>
-        </geometry>
-        <material name="LightGrey">
-          <color rgba="0.7 0.7 0.7 1.0"/>
-        </material>
-      </visual>
-      <collision>
-        <geometry>
-          <mesh filename="package://shallow_depth_insertion_v2/meshes/ur10/collision/base.stl"/>
+          <mesh filename="package://shallow_depth_insertion/meshes/ur10/visual/base.dae"/>
+        </geometry>
+        <material name="LightGrey">
+          <color rgba="0.7 0.7 0.7 1.0"/>
+        </material>
+      </visual>
+      <collision>
+        <geometry>
+          <mesh filename="package://shallow_depth_insertion/meshes/ur10/collision/base.stl"/>
         </geometry>
       </collision>
@@ -93,13 +93,13 @@
       <visual>
         <geometry>
-          <mesh filename="package://shallow_depth_insertion_v2/meshes/ur10/visual/shoulder.dae"/>
-        </geometry>
-        <material name="LightGrey">
-          <color rgba="0.7 0.7 0.7 1.0"/>
-        </material>
-      </visual>
-      <collision>
-        <geometry>
-          <mesh filename="package://shallow_depth_insertion_v2/meshes/ur10/collision/shoulder.stl"/>
+          <mesh filename="package://shallow_depth_insertion/meshes/ur10/visual/shoulder.dae"/>
+        </geometry>
+        <material name="LightGrey">
+          <color rgba="0.7 0.7 0.7 1.0"/>
+        </material>
+      </visual>
+      <collision>
+        <geometry>
+          <mesh filename="package://shallow_depth_insertion/meshes/ur10/collision/shoulder.stl"/>
         </geometry>
       </collision>
@@ -124,13 +124,13 @@
       <visual>
         <geometry>
-          <mesh filename="package://shallow_depth_insertion_v2/meshes/ur10/visual/upperarm.dae"/>
-        </geometry>
-        <material name="LightGrey">
-          <color rgba="0.7 0.7 0.7 1.0"/>
-        </material>
-      </visual>
-      <collision>
-        <geometry>
-          <mesh filename="package://shallow_depth_insertion_v2/meshes/ur10/collision/upperarm.stl"/>
+          <mesh filename="package://shallow_depth_insertion/meshes/ur10/visual/upperarm.dae"/>
+        </geometry>
+        <material name="LightGrey">
+          <color rgba="0.7 0.7 0.7 1.0"/>
+        </material>
+      </visual>
+      <collision>
+        <geometry>
+          <mesh filename="package://shallow_depth_insertion/meshes/ur10/collision/upperarm.stl"/>
         </geometry>
       </collision>
@@ -155,13 +155,13 @@
       <visual>
          <geometry>
-          <mesh filename="package://shallow_depth_insertion_v2/meshes/ur10/visual/forearm.dae"/>
-        </geometry>
-        <material name="LightGrey">
-          <color rgba="0.7 0.7 0.7 1.0"/>
-        </material>
-      </visual>
-      <collision>
-        <geometry>
-          <mesh filename="package://shallow_depth_insertion_v2/meshes/ur10/collision/forearm.stl"/>
+          <mesh filename="package://shallow_depth_insertion/meshes/ur10/visual/forearm.dae"/>
+        </geometry>
+        <material name="LightGrey">
+          <color rgba="0.7 0.7 0.7 1.0"/>
+        </material>
+      </visual>
+      <collision>
+        <geometry>
+          <mesh filename="package://shallow_depth_insertion/meshes/ur10/collision/forearm.stl"/>
         </geometry>
       </collision>
@@ -186,13 +186,13 @@
       <visual>
         <geometry>
-          <mesh filename="package://shallow_depth_insertion_v2/meshes/ur10/visual/wrist1.dae"/>
-        </geometry>
-        <material name="LightGrey">
-          <color rgba="0.7 0.7 0.7 1.0"/>
-        </material>
-      </visual>
-      <collision>
-        <geometry>
-          <mesh filename="package://shallow_depth_insertion_v2/meshes/ur10/collision/wrist1.stl"/>
+          <mesh filename="package://shallow_depth_insertion/meshes/ur10/visual/wrist1.dae"/>
+        </geometry>
+        <material name="LightGrey">
+          <color rgba="0.7 0.7 0.7 1.0"/>
+        </material>
+      </visual>
+      <collision>
+        <geometry>
+          <mesh filename="package://shallow_depth_insertion/meshes/ur10/collision/wrist1.stl"/>
         </geometry>
       </collision>
@@ -217,13 +217,13 @@
       <visual>
         <geometry>
-          <mesh filename="package://shallow_depth_insertion_v2/meshes/ur10/visual/wrist2.dae"/>
-        </geometry>
-        <material name="LightGrey">
-          <color rgba="0.7 0.7 0.7 1.0"/>
-        </material>
-      </visual>
-      <collision>
-        <geometry>
-          <mesh filename="package://shallow_depth_insertion_v2/meshes/ur10/collision/wrist2.stl"/>
+          <mesh filename="package://shallow_depth_insertion/meshes/ur10/visual/wrist2.dae"/>
+        </geometry>
+        <material name="LightGrey">
+          <color rgba="0.7 0.7 0.7 1.0"/>
+        </material>
+      </visual>
+      <collision>
+        <geometry>
+          <mesh filename="package://shallow_depth_insertion/meshes/ur10/collision/wrist2.stl"/>
         </geometry>
       </collision>
@@ -248,13 +248,13 @@
       <visual>
         <geometry>
-          <mesh filename="package://shallow_depth_insertion_v2/meshes/ur10/visual/wrist3.dae"/>
-        </geometry>
-        <material name="LightGrey">
-          <color rgba="0.7 0.7 0.7 1.0"/>
-        </material>
-      </visual>
-      <collision>
-        <geometry>
-          <mesh filename="package://shallow_depth_insertion_v2/meshes/ur10/collision/wrist3.stl"/>
+          <mesh filename="package://shallow_depth_insertion/meshes/ur10/visual/wrist3.dae"/>
+        </geometry>
+        <material name="LightGrey">
+          <color rgba="0.7 0.7 0.7 1.0"/>
+        </material>
+      </visual>
+      <collision>
+        <geometry>
+          <mesh filename="package://shallow_depth_insertion/meshes/ur10/collision/wrist3.stl"/>
         </geometry>
       </collision>

File: urdf/ur10_joint_limited_robot.urdf.xacro (robot description, xacro)
@@ -3,12 +3,12 @@
        name="ur10" >
   <!-- common stuff -->
-  <xacro:include filename="$(find shallow_depth_insertion_v2)/urdf/common.gazebo.xacro" />
+  <xacro:include filename="$(find shallow_depth_insertion)/urdf/common.gazebo.xacro" />
   <!-- ur10 -->
-  <xacro:include filename="$(find shallow_depth_insertion_v2)/urdf/ur10.urdf.xacro" />
+  <xacro:include filename="$(find shallow_depth_insertion)/urdf/ur10.urdf.xacro" />
   <!-- gripper -->
-  <xacro:include filename="$(find shallow_depth_insertion_v2)/urdf/robotiq_arg2f_140_model/robotiq_arg2f_140_model_macro.xacro" />
+  <xacro:include filename="$(find shallow_depth_insertion)/urdf/robotiq_arg2f_140_model/robotiq_arg2f_140_model_macro.xacro" />
   <xacro:robotiq_arg2f_140 prefix=""/>
   <!-- ft sensor -->
-  <xacro:include filename="$(find shallow_depth_insertion_v2)/urdf/robotiq_ft_sensor/robotiq_ft300.urdf.xacro" />
+  <xacro:include filename="$(find shallow_depth_insertion)/urdf/robotiq_ft_sensor/robotiq_ft300.urdf.xacro" />
   <!-- arm -->
   <xacro:ur10_robot prefix="" joint_limited="true"

File: urdf/ur10_robot.urdf.xacro (robot description, xacro)
@@ -3,9 +3,9 @@
        name="ur10" >
   <!-- common stuff -->
-  <xacro:include filename="$(find shallow_depth_insertion_v2)/urdf/common.gazebo.xacro" />
+  <xacro:include filename="$(find shallow_depth_insertion)/urdf/common.gazebo.xacro" />
   <!-- ur10 -->
-  <xacro:include filename="$(find shallow_depth_insertion_v2)/urdf/ur10_robotiq2f140mm.urdf.xacro" />
+  <xacro:include filename="$(find shallow_depth_insertion)/urdf/ur10_robotiq2f140mm.urdf.xacro" />
   <!-- gripper -->
-  <xacro:include filename="$(find shallow_depth_insertion_v2)/urdf/robotiq_arg2f_140_model/robotiq_arg2f_140_model_macro.xacro" />
+  <xacro:include filename="$(find shallow_depth_insertion)/urdf/robotiq_arg2f_140_model/robotiq_arg2f_140_model_macro.xacro" />
   <xacro:robotiq_arg2f_140 prefix=""/>
   <!-- ft sensor -->
