Commit message: gripper simulation

File: urdf/robotiq_arg2f_140_model/robotiq_arg2f_140_model_macro.xacro (robot description, xacro)
@@ -160,5 +160,5 @@
       <axis xyz="1 0 0" />
       <limit lower="-0.8757" upper="0.8757" velocity="2.0" effort="1000" />
-      <mimic joint="${prefix}finger_joint" multiplier="-1" offset="0" />
+      <mimic joint="${prefix}gripper_finger_joint" multiplier="-1" offset="0" />
     </joint>
   </xacro:macro>
@@ -170,7 +170,20 @@
       <axis xyz="1 0 0" />
       <limit lower="-0.8757" upper="0.8757" velocity="2.0" effort="1000" />
-      <mimic joint="${prefix}finger_joint" multiplier="1" offset="0" />
-    </joint>
-  </xacro:macro>
+      <mimic joint="${prefix}gripper_finger_joint" multiplier="1" offset="0" />
+    </joint>
+  </xacro:macro>
+  <!--JOHN-->
+  <xacro:macro name="left_outer_knuckle_joint" params="prefix">
+    <joint name="${prefix}left_outer_knuckle_joint" type="revolute">
+      <origin xyz="0 0.030601 0.054905" rpy="${pi / 2 + .725} 0 ${pi}" />
+      <parent link="${prefix}robotiq_arg2f_base_link" />
+      <child link="${prefix}left_outer_knuckle" />
+      <axis xyz="1 0 0" />
+      <limit lower="-0.725" upper="0.725" velocity="2.0" effort="1000" />
+    <mimic joint="${prefix}gripper_finger_joint" multiplier="-1" offset="0" />
+    </joint>
+    <xacro:finger_joints prefix="${prefix}" fingerprefix="left" reflect="1.0"/>
+  </xacro:macro>
+  <!--JOHN-->
   <xacro:macro name="inner_finger_pad_joint" params="prefix fingerprefix">
     <joint name="${prefix}${fingerprefix}_inner_finger_pad_joint" type="fixed">
@@ -189,4 +202,5 @@
       <axis xyz="-1 0 0" />
       <limit lower="0" upper="0.7" velocity="2.0" effort="1000" />
+      <mimic joint="gripper_finger_joint" multiplier="1.0" offset="0.0" />
     </joint>
     <xacro:finger_joints prefix="${prefix}" fingerprefix="left" reflect="1.0"/>
@@ -199,5 +213,5 @@
       <axis xyz="1 0 0" />
       <limit lower="-0.725" upper="0.725" velocity="2.0" effort="1000" />
-    <mimic joint="${prefix}finger_joint" multiplier="-1" offset="0" />
+    <mimic joint="${prefix}gripper_finger_joint" multiplier="-1" offset="0" />
     </joint>
     <xacro:finger_joints prefix="${prefix}" fingerprefix="right" reflect="-1.0"/>
@@ -211,3 +225,19 @@
     <xacro:robotiq_arg2f_transmission prefix="${prefix}"/>
   </xacro:macro>
+  <!-- Indirect Joint to Visualize Gripper movement by John -->
+  <link name="temp">
+    <visual>
+      <origin xyz="0 0 0" rpy="0 0 0" />
+      <geometry>
+        <box size="0.0 0.0 0.0"/>
+      </geometry>
+    </visual>
+  </link>
+  <joint name="gripper_finger_joint" type="revolute">
+    <origin xyz="0 0 0" rpy="0 0 0" />
+    <parent link="world" />
+    <child link="temp" />
+    <axis xyz="1 0 0" />
+    <limit lower="0" upper="0.7" velocity="2.0" effort="1000" />
+  </joint>
 </robot>

File: urdf/robotiq_ft_sensor/robotiq_ft300.urdf.xacro (robot description, xacro)
@@ -30,5 +30,5 @@
                 <origin xyz="0 0 0" rpy="0 0 0" />
                 <geometry>
-                    <mesh filename="package://robotiq_ft_sensor/meshes/visual/robotiq_ft300.STL"/>
+                    <mesh filename="package://shallow_depth_insertion_v2/meshes/robotiq_ft_sensor/visual/robotiq_ft300.STL"/>
                 </geometry>
                 <material name="Robotiq-Black">
@@ -39,5 +39,5 @@
                 <origin xyz="0 0 0" rpy="0 0 0" />
                 <geometry>
-                    <mesh filename="package://robotiq_ft_sensor/meshes/collision/robotiq_ft300.STL"/>
+                    <mesh filename="package://shallow_depth_insertion_v2/meshes/robotiq_ft_sensor/collision/robotiq_ft300.STL"/>
                 </geometry>
             </collision>
@@ -48,5 +48,5 @@
                 <origin xyz="0 0 0" rpy="0 0 0" />
                 <geometry>
-                    <mesh filename="package://robotiq_ft_sensor/meshes/visual/mountings/robotiq_ft300-G-062-COUPLING_G-50-4M6-1D6_20181119.STL"/>
+                    <mesh filename="package://shallow_depth_insertion_v2/meshes/robotiq_ft_sensor/visual/mountings/robotiq_ft300-G-062-COUPLING_G-50-4M6-1D6_20181119.STL"/>
                 </geometry>
                 <material name="Robotiq-Grey">
@@ -57,5 +57,5 @@
                 <origin xyz="0 0 0" rpy="0 0 0" />
                 <geometry>
-                    <mesh filename="package://robotiq_ft_sensor/meshes/collision/mountings/robotiq_ft300-G-062-COUPLING_G-50-4M6-1D6_20181119.STL"/>
+                    <mesh filename="package://shallow_depth_insertion_v2/meshes/robotiq_ft_sensor/collision/mountings/robotiq_ft300-G-062-COUPLING_G-50-4M6-1D6_20181119.STL"/>
                 </geometry>
             </collision>

File: urdf/robotiq_ft_sensor/robotiq_fts150.urdf.xacro (robot description, xacro)
@@ -18,5 +18,5 @@
                 <origin xyz="0 0 0" rpy="0 0 0" />
                 <geometry>
-                    <mesh filename="package://robotiq_ft_sensor/meshes/visual/robotiq_fts150.stl"/>
+                    <mesh filename="package://shallow_depth_insertion_v2/meshes/robotiq_ft_sensor/visual/robotiq_fts150.stl"/>
                 </geometry>
                 <material name="black"/>
@@ -25,5 +25,5 @@
                 <origin xyz="0 0 0" rpy="0 0 0" />
                 <geometry>
-                    <mesh filename="package://robotiq_ft_sensor/meshes/collision/robotiq_fts150.stl"/>
+                    <mesh filename="package://shallow_depth_insertion_v2/meshes/robotiq_ft_sensor/collision/robotiq_fts150.stl"/>
                 </geometry>
             </collision>

File: urdf/ur10_joint_limited_robot.urdf.xacro (robot description, xacro)
@@ -7,8 +7,8 @@
   <xacro:include filename="$(find shallow_depth_insertion_v2)/urdf/ur10.urdf.xacro" />
   <!-- gripper -->
-  <!--xacro:include filename="$(find shallow_depth_insertion_v2)/urdf/robotiq_arg2f_140_model/robotiq_arg2f_140_model_macro.xacro" />
-  <xacro:robotiq_arg2f_140 prefix=""/-->
+  <xacro:include filename="$(find shallow_depth_insertion_v2)/urdf/robotiq_arg2f_140_model/robotiq_arg2f_140_model_macro.xacro" />
+  <xacro:robotiq_arg2f_140 prefix=""/>
   <!-- ft sensor -->
-  <!--xacro:include filename="$(find robotiq_ft_sensor)/urdf/robotiq_ft300.urdf.xacro" /-->
+  <xacro:include filename="$(find shallow_depth_insertion_v2)/urdf/robotiq_ft_sensor/robotiq_ft300.urdf.xacro" />
   <!-- arm -->
   <xacro:ur10_robot prefix="" joint_limited="true"
@@ -26,11 +26,11 @@
     <origin xyz="0.0 0.0 0.0" rpy="0.0 0.0 0.0" />
   </joint>
-  <!--xacro:robotiq_ft300 parent="ee_link" prefix="">
+  <xacro:robotiq_ft300 parent="ee_link" prefix="">
 		<origin xyz="-0.01 0.0 0.0" rpy="3.14159265359 -1.57079632679 0.0"/>
-	</xacro:robotiq_ft300-->
-  <!--joint name="gripper2sensor" type="fixed">
+	</xacro:robotiq_ft300>
+  <joint name="gripper2sensor" type="fixed">
     <parent link="robotiq_ft_frame_id" />
     <child link = "robotiq_arg2f_base_link" />
     <origin xyz="0.0 0.0 -0.0065" rpy="0.0 0.0 0.0" />
-  </joint-->
+  </joint>
 </robot>

Commit message: changed urdf to visualize gripper

File: urdf/robotiq_arg2f_140_model/robotiq_arg2f_140_model_macro.xacro (robot description, xacro)
@@ -173,17 +173,4 @@
     </joint>
   </xacro:macro>
-  <!--JOHN-->
-  <xacro:macro name="left_outer_knuckle_joint" params="prefix">
-    <joint name="${prefix}left_outer_knuckle_joint" type="revolute">
-      <origin xyz="0 0.030601 0.054905" rpy="${pi / 2 + .725} 0 ${pi}" />
-      <parent link="${prefix}robotiq_arg2f_base_link" />
-      <child link="${prefix}left_outer_knuckle" />
-      <axis xyz="1 0 0" />
-      <limit lower="-0.725" upper="0.725" velocity="2.0" effort="1000" />
-    <mimic joint="${prefix}gripper_finger_joint" multiplier="-1" offset="0" />
-    </joint>
-    <xacro:finger_joints prefix="${prefix}" fingerprefix="left" reflect="1.0"/>
-  </xacro:macro>
-  <!--JOHN-->
   <xacro:macro name="inner_finger_pad_joint" params="prefix fingerprefix">
     <joint name="${prefix}${fingerprefix}_inner_finger_pad_joint" type="fixed">
@@ -196,5 +183,5 @@
   <xacro:include filename="$(find shallow_depth_insertion)/urdf/robotiq_arg2f_140_model/robotiq_arg2f.xacro" />
   <xacro:macro name="finger_joint" params="prefix">
-    <joint name="${prefix}finger_joint" type="revolute">
+    <joint name="${prefix}my_finger_joint" type="revolute">
       <origin xyz="0 -0.030601 0.054905" rpy="${pi / 2 + .725} 0 0" />
       <parent link="${prefix}robotiq_arg2f_base_link" />
@@ -226,5 +213,5 @@
   </xacro:macro>
   <!-- Indirect Joint to Visualize Gripper movement by John -->
-  <link name="temp">
+  <link name="temp1">
     <visual>
       <origin xyz="0 0 0" rpy="0 0 0" />
@@ -237,7 +224,31 @@
     <origin xyz="0 0 0" rpy="0 0 0" />
     <parent link="world" />
-    <child link="temp" />
+    <child link="temp1" />
     <axis xyz="1 0 0" />
     <limit lower="0" upper="0.7" velocity="2.0" effort="1000" />
   </joint>
+  <link name="temp2">
+    <visual>
+      <geometry>
+        <box size="0.01 0.01 0.01"/>
+      </geometry>
+      <origin rpy="0 0 0" xyz="0 0 0"/>
+    </visual>
+    <inertial>
+      <origin xyz="0 0 0" rpy="0 0 0" />
+      <mass value="1" />
+      <inertia
+        ixx="1.0" ixy="0.0" ixz="0.0"
+        iyy="1.0" iyz="0.0"
+        izz="1.0" />
+    </inertial>
+  </link>
+  <joint name="finger_joint" type="revolute">
+    <origin xyz="0 0 0" rpy="0 0 0" />
+    <parent link="world" />
+    <child link="temp2" />
+    <axis xyz="1 0 0" />
+    <limit lower="0" upper="0.7" velocity="2.0" effort="1000" />
+  </joint>
+  <!-- Indirect Joint to Visualize Gripper movement by John -->
 </robot>

File: urdf/ur10_joint_limited_robot.urdf.xacro (robot description, xacro)
@@ -19,5 +19,5 @@
 		 wrist_2_lower_limit="${-pi}" wrist_2_upper_limit="${pi}"
 		 wrist_3_lower_limit="${-pi}" wrist_3_upper_limit="${pi}"
-/>
+  />
   <link name="world" />
   <joint name="world_joint" type="fixed">
@@ -34,3 +34,38 @@
     <origin xyz="0.0 0.0 -0.0065" rpy="0.0 0.0 0.0" />
   </joint>
+  <!-- environment -->
+  <material name="white">
+    <color rgba="1 1 1 1"/>
+  </material>
+  <material name="blue">
+    <color rgba="0 0 0.8 1"/>
+  </material>
+  <link name="robot_platform">
+    <visual>
+      <geometry>
+        <box size="0.25 0.25 0.02"/>
+      </geometry>
+      <origin rpy="0 0 0" xyz="0 0 -0.01"/>
+      <material name="white"/>
+    </visual>
+  </link>
+  <joint name="robot_to_robot_platform" type="fixed">
+    <parent link="base_link"/>
+    <child link="robot_platform"/>
+    <origin xyz="0 0 0"/>
+  </joint>
+  <link name="table">
+    <visual>
+      <geometry>
+        <box size="1.8 2.4 0.1"/>
+      </geometry>
+      <origin rpy="0 0 0" xyz="0.64 -0.94 -0.05"/>
+      <material name="white"/>
+    </visual>
+  </link>
+  <joint name="robot_platform_to_table" type="fixed">
+    <parent link="robot_platform"/>
+    <child link="table"/>
+    <origin xyz="0 0 -0.02"/>
+  </joint>
 </robot>
