Commit message: update README.md

File: urdf/ur10_joint_limited_robot.urdf.xacro (robot description, xacro)
@@ -7,8 +7,8 @@
   <xacro:include filename="$(find shallow_depth_insertion_v2)/urdf/ur10.urdf.xacro" />
   <!-- gripper -->
-  <xacro:include filename="$(find shallow_depth_insertion_v2)/urdf/robotiq_arg2f_140_model/robotiq_arg2f_140_model_macro.xacro" />
-  <xacro:robotiq_arg2f_140 prefix=""/>
+  <!--xacro:include filename="$(find shallow_depth_insertion_v2)/urdf/robotiq_arg2f_140_model/robotiq_arg2f_140_model_macro.xacro" />
+  <xacro:robotiq_arg2f_140 prefix=""/-->
   <!-- ft sensor -->
-  <xacro:include filename="$(find robotiq_ft_sensor)/urdf/robotiq_ft300.urdf.xacro" />
+  <!--xacro:include filename="$(find robotiq_ft_sensor)/urdf/robotiq_ft300.urdf.xacro" /-->
   <!-- arm -->
   <xacro:ur10_robot prefix="" joint_limited="true"
@@ -26,11 +26,11 @@
     <origin xyz="0.0 0.0 0.0" rpy="0.0 0.0 0.0" />
   </joint>
-  <xacro:robotiq_ft300 parent="ee_link" prefix="">
+  <!--xacro:robotiq_ft300 parent="ee_link" prefix="">
 		<origin xyz="-0.01 0.0 0.0" rpy="3.14159265359 -1.57079632679 0.0"/>
-	</xacro:robotiq_ft300>
-  <joint name="gripper2sensor" type="fixed">
+	</xacro:robotiq_ft300-->
+  <!--joint name="gripper2sensor" type="fixed">
     <parent link="robotiq_ft_frame_id" />
     <child link = "robotiq_arg2f_base_link" />
     <origin xyz="0.0 0.0 -0.0065" rpy="0.0 0.0 0.0" />
-  </joint>
+  </joint-->
 </robot>

Commit message: hardware test successful

File: urdf/ur10_joint_limited_robot.urdf.xacro (robot description, xacro)
@@ -60,5 +60,5 @@
         <box size="1.8 2.4 0.1"/>
       </geometry>
-      <origin rpy="0 0 0" xyz="0.64 -0.94 -0.05"/>
+      <origin rpy="0 0 0" xyz="-0.64 0.94 -0.05"/>
       <material name="white"/>
     </visual>

Commit message: object visual during regrasp

File: urdf/ur10_joint_limited_robot.urdf.xacro (robot description, xacro)
@@ -32,5 +32,5 @@
     <parent link="robotiq_ft_frame_id" />
     <child link = "robotiq_arg2f_base_link" />
-    <origin xyz="0.0 0.0 -0.0065" rpy="0.0 0.0 0.0" />
+    <origin xyz="0.0 0.0 -0.001" rpy="0.0 0.0 -1.57079632679" />
   </joint>
   <!-- environment -->

Commit message: SDI_main_sim.py complete

File: urdf/ur10_joint_limited_robot.urdf.xacro (robot description, xacro)
@@ -32,5 +32,6 @@
     <parent link="robotiq_ft_frame_id" />
     <child link = "robotiq_arg2f_base_link" />
-    <origin xyz="0.0 0.0 -0.001" rpy="0.0 0.0 -1.57079632679" />
+    <origin xyz="0.0 0.0 0.016" rpy="0.0 0.0 -1.57079632679" />
+    <!--origin xyz="0.0 0.0 -0.0065" rpy="0.0 0.0 0.0" /-->
   </joint>
   <!-- environment -->

Commit message: Add sliding release and generalized release function

File: urdf/ur10_joint_limited_robot.urdf.xacro (robot description, xacro)
@@ -56,4 +56,5 @@
     <origin xyz="0 0 0"/>
   </joint>
+  <!--
   <link name="table">
     <visual>
@@ -65,4 +66,15 @@
     </visual>
   </link>
+  -->
+  <!--new table setup-->
+  <link name="table">
+    <visual>
+      <geometry>
+        <box size="1.8 1.2 0.1"/>
+      </geometry>
+      <origin rpy="0 0 0" xyz="-0.08 -0.44 -0.05"/>
+      <material name="white"/>
+    </visual>
+  </link>
   <joint name="robot_platform_to_table" type="fixed">
     <parent link="robot_platform"/>
@@ -70,3 +82,32 @@
     <origin xyz="0 0 -0.02"/>
   </joint>
+  <!--protection wall-->
+  <link name="wall1">
+    <visual>
+      <geometry>
+        <box size="1.8 0.1 1.5"/>
+      </geometry>
+      <origin rpy="0 0 0" xyz="-0.08 0.21 0.75"/>
+      <material name="white"/>
+    </visual>
+  </link>
+  <joint name="table_to_wall1" type="fixed">
+    <parent link="table"/>
+    <child link="wall1"/>
+    <origin xyz="0 0 0"/>
+  </joint>
+  <link name="wall2">
+    <visual>
+      <geometry>
+        <box size="0.1 1.2 1.5"/>
+      </geometry>
+      <origin rpy="0 0 0" xyz="0.87 -0.44 0.75"/>
+      <material name="white"/>
+    </visual>
+  </link>
+  <joint name="table_to_wall2" type="fixed">
+    <parent link="table"/>
+    <child link="wall2"/>
+    <origin xyz="0 0 0"/>
+  </joint>
 </robot>

Commit message: code backup

File: urdf/ur10_joint_limited_robot.urdf.xacro (robot description, xacro)
@@ -97,5 +97,5 @@
     <origin xyz="0 0 0"/>
   </joint>
-  <link name="wall2">
+  <!-- <link name="wall2">
     <visual>
       <geometry>
@@ -110,4 +110,4 @@
     <child link="wall2"/>
     <origin xyz="0 0 0"/>
-  </joint>
+  </joint> -->
 </robot>
